File: 4in1ESC.kicad_pcb (KiCad board)
At the start: 6 copper layers, 31.2 x 33 mm, 206 parts, among them Q1 SP40N03GNJ, Q10 SP40N03GNJ, Q11 SP40N03GNJ, Q12 SP40N03GNJ, Q13 SP40N03GNJ, Q14 SP40N03GNJ, Q15 SP40N03GNJ, Q16 SP40N03GNJ, Q17 SP40N03GNJ, Q18 SP40N03GNJ, Q19 SP40N03GNJ, Q2 SP40N03GNJ, Q20 SP40N03GNJ, Q21 SP40N03GNJ, Q22 SP40N03GNJ, Q23 SP40N03GNJ, Q24 SP40N03GNJ, Q3 SP40N03GNJ, Q4 SP40N03GNJ, Q5 SP40N03GNJ, Q6 SP40N03GNJ, Q7 SP40N03GNJ, Q8 SP40N03GNJ, Q9 SP40N03GNJ, U1 INA199A1DCKR, U10 AT32F421G8U7, U11 NSG2065Q, U14 HC-1_0-8PWT, U18 LMR51420YDDCR, U2 AT32F421G8U7, U26 TPS746-3.3DRV, U3 NSG2065Q, U5 XRIM160808SR47MBCD, U6 AT32F421G8U7, U7 NSG2065Q, U8 AT32F421G8U7, U9 NSG2065Q

Commit message: Replaced the old ESC Connector with JST-SH series
Parts:
- removed U14: HC-1_0-8PWT, components:CONN-SMD_HC-1.0-8PWT
- added J1: SM08B-SRSS-TB, Connector_JST:JST_SH_SM08B-SRSS-TB_1x08-1MP_P1.00mm_Horizontal, B.Cu at (76.0, 35.8)
- moved C55 9.40 mm to (75.5, 16.9)
- moved C56 9.40 mm to (75.5, 19.9)
- moved C58 9.40 mm to (75.5, 22.9)
- moved C60 9.40 mm to (80.0, 16.9)
- moved C61 9.40 mm to (80.0, 19.9)
- moved C62 9.40 mm to (80.0, 22.9)
- moved C30 9.40 mm to (71.0, 16.9)
- moved C52 9.40 mm to (71.0, 19.9)
- moved C54 9.40 mm to (71.0, 22.9)
Connections:
- U4 pad 10: GND -> /M4
- U4 pad 3: /CURR -> +BATT
- U4 pad 4: unconnected-(U4-T-Pad4) -> GND
- U4 pad 5: /M4 -> /CURR
- U4 pad 6: /M3 -> unconnected-(U4-TX-Pad6)
- U4 pad 7: /M2 -> /M1
- U4 pad 8: /M1 -> /M2
- U4 pad 9: +BATT -> /M3
Routing:
- net GND: track 90.1 -> 68.6 mm, vias 189 -> 177
- net /M4: track 7.85 -> 25.7 mm, vias 1 -> 2
- net /M3: track 10.9 -> 14.8 mm, vias 1 -> 2
- net /M1: track 6.36 -> 9.53 mm
- net +BATT: track 16.0 -> 17.7 mm, vias 11 -> 20
- net /M2: track 7.93 -> 6.82 mm
- net /CURR: track 7.67 -> 8.61 mm
- net Net-(Q8-G): track 20.4 -> 19.9 mm
- net unconnected-(U4-TX-Pad6): vias 0 -> 1
- added copper zone on B.Cu, net +BATT
Other:
- board text added: "+ - C T"
- board text added: "+ -C T 1 2 3 4"
- board text added: "1 2 3 4"
- board text removed: "- + 1 2"
- board text removed: "3 4 T C"
- board text removed: "C T 4 3 2 1 + -"
