File: 4in1ESC.kicad_pcb (KiCad board)
At the start: 6 copper layers, 31.2 x 33 mm, 206 parts, among them J1 SM08B-SRSS-TB, Q1 SP40N03GNJ, Q10 SP40N03GNJ, Q11 SP40N03GNJ, Q12 SP40N03GNJ, Q13 SP40N03GNJ, Q14 SP40N03GNJ, Q15 SP40N03GNJ, Q16 SP40N03GNJ, Q17 SP40N03GNJ, Q18 SP40N03GNJ, Q19 SP40N03GNJ, Q2 SP40N03GNJ, Q20 SP40N03GNJ, Q21 SP40N03GNJ, Q22 SP40N03GNJ, Q23 SP40N03GNJ, Q24 SP40N03GNJ, Q3 SP40N03GNJ, Q4 SP40N03GNJ, Q5 SP40N03GNJ, Q6 SP40N03GNJ, Q7 SP40N03GNJ, Q8 SP40N03GNJ, Q9 SP40N03GNJ, U1 INA199A1DCKR, U10 AT32F421G8U7, U11 NSG2065Q, U18 LMR51420YDDCR, U2 AT32F421G8U7, U26 TPS746-3.3DRV, U3 NSG2065Q, U5 XRIM160808SR47MBCD, U6 AT32F421G8U7, U7 NSG2065Q, U8 AT32F421G8U7, U9 NSG2065Q

Commit message: Added many compatibilty and fixed all issues, ready for ordering V1
Parts:
- removed C30, C52, C54, C55, C56, C58, C60, C61, C62: 10uF, Capacitor_SMD:C_0805_2012Metric
- removed U26: TPS746-3.3DRV, Package_SON:WSON-6-1EP_2x2mm_P0.65mm_EP1x1.6mm
- added U12: INA186A3IDCKR, 4in1ESC:SOT-363_SC-70-6, B.Cu at (76.0, 57.4)
- FB1, FB2, FB3, FB4: value 200mA -> BLM03PX121SN1D
- J1: footprint Connector_JST:JST_SH_SM08B-SRSS-TB_1x08-1MP_P1.00mm_Horizontal -> 4in1ESC:JST_SM08B-SRSS-TB
- U1: value INA199A1DCKR -> TLV76733DRVR; footprint Package_TO_SOT_SMD:SOT-363_SC-70-6 -> 4in1ESC:WSON-6_L2.0-W2.0-P0.65-TL-EP
- moved U1 13.5 mm to (75.6, 43.9), turned to -90 degrees
- moved C49 6.48 mm to (78.4, 49.7)
- moved C48 6.10 mm to (84.8, 49.9), turned to 90 degrees
- moved C70 3.46 mm to (74.6, 46.2), turned to -90 degrees
- moved J1 2.77 mm to (76.0, 33.0)
- moved C43 0.55 mm to (76.0, 47.0), turned to 45 degrees
- moved FB2 0.48 mm to (79.0, 49.7), turned to -90 degrees
- moved C46 0.09 mm to (78.7, 43.7)
Connections:
- R73 pad 2: Net-(U1-OUT) -> Net-(U12-OUT)
- Rsense1 pad 1: Net-(U1-+) -> /CSA+
- U1 pad 2: GND -> +3V3
- U1 pad 3: +3V3 -> GND
- U1 pad 4: Net-(U1-+) -> +8V
- U1 pad 5: +BATT -> GND
- U1 pad 6: Net-(U1-OUT) -> +8V
- U4 pad 1: Net-(U1-+) -> /CSA+
Routing:
- net Net-(U12-OUT): track 0.00 -> 20.4 mm, vias 0 -> 2
- net Net-(U1-OUT): track 20.0 -> 0.00 mm, vias 2 -> 0
- net GND: track 68.6 -> 74.2 mm, vias 177 -> 176
- net +3V3: track 76.9 -> 81.4 mm
- net +8V: track 9.35 -> 13.5 mm
- net Net-(U1-+): track 3.69 -> 0.00 mm, vias 29 -> 0
- net /CSA+: track 0.00 -> 3.69 mm, vias 0 -> 29
- net Net-(U2-PB4): track 15.5 -> 14.7 mm
- net /M4: track 25.7 -> 25.0 mm
- added copper zone on F.Cu, net /CSA+
- removed copper zone on F.Cu, net Net-(U1-+)

Commit message: final layout
Connections:
- U1 pad 1: GND -> +3V3
Routing:
- net +3V3: track 81.4 -> 83.1 mm
- net GND: track 74.2 -> 73.6 mm
Other:
- board text added: "ESC"
- board text added: "open"
- board text removed: "V0.1"
