File: 4in1ESC.kicad_pcb (KiCad board)
At the start: 6 copper layers, 31.2 x 33 mm, 197 parts, among them J1 SM08B-SRSS-TB, Q1 SP40N03GNJ, Q10 SP40N03GNJ, Q11 SP40N03GNJ, Q12 SP40N03GNJ, Q13 SP40N03GNJ, Q14 SP40N03GNJ, Q15 SP40N03GNJ, Q16 SP40N03GNJ, Q17 SP40N03GNJ, Q18 SP40N03GNJ, Q19 SP40N03GNJ, Q2 SP40N03GNJ, Q20 SP40N03GNJ, Q21 SP40N03GNJ, Q22 SP40N03GNJ, Q23 SP40N03GNJ, Q24 SP40N03GNJ, Q3 SP40N03GNJ, Q4 SP40N03GNJ, Q5 SP40N03GNJ, Q6 SP40N03GNJ, Q7 SP40N03GNJ, Q8 SP40N03GNJ, Q9 SP40N03GNJ, U1 TLV76733DRVR, U10 AT32F421G8U7, U11 NSG2065Q, U12 INA186A3IDCKR, U18 LMR51420YDDCR, U2 AT32F421G8U7, U3 NSG2065Q, U5 XRIM160808SR47MBCD, U6 AT32F421G8U7, U7 NSG2065Q, U8 AT32F421G8U7, U9 NSG2065Q

Commit message: Standardize repo: .gitignore, README, license, remove production from tracking
- Standardize .gitignore to match ecosystem template
- Update README: fix production refs, add missing dirs, simplify license section
- Replace LICENSE stub with full CERN-OHL-S-2.0 text
- Remove production/ from git tracking (generated, re-exportable)
- Add previously untracked: licensing/, COST_ANALYSIS.md, tools/esc_thermal.py
- Delete NextPCB artifact (bom_template_nextpcb)

Co-Authored-By: Claude Opus 4.6 (1M context) <noreply@anthropic.com>
Parts:
- FB1, FB2, FB3, FB4: value BLM03PX121SN1D -> BLM03HD331SN1D
