File: _autosave-4in1ESC.kicad_pcb (KiCad board)
At the start: 6 copper layers, 31.2 x 33 mm, 206 parts, among them J1 SM08B-SRSS-TB, Q1 SP40N03GNJ, Q10 SP40N03GNJ, Q11 SP40N03GNJ, Q12 SP40N03GNJ, Q13 SP40N03GNJ, Q14 SP40N03GNJ, Q15 SP40N03GNJ, Q16 SP40N03GNJ, Q17 SP40N03GNJ, Q18 SP40N03GNJ, Q19 SP40N03GNJ, Q2 SP40N03GNJ, Q20 SP40N03GNJ, Q21 SP40N03GNJ, Q22 SP40N03GNJ, Q23 SP40N03GNJ, Q24 SP40N03GNJ, Q3 SP40N03GNJ, Q4 SP40N03GNJ, Q5 SP40N03GNJ, Q6 SP40N03GNJ, Q7 SP40N03GNJ, Q8 SP40N03GNJ, Q9 SP40N03GNJ, U1 TLV76733DRVR, U10 AT32F421G8U7, U11 NSG2065Q, U12 INA186A3IDCKR, U18 LMR51420YDDCR, U2 AT32F421G8U7, U3 NSG2065Q, U5 XRIM160808SR47MBCD, U6 AT32F421G8U7, U7 NSG2065Q, U8 AT32F421G8U7, U9 NSG2065Q

Commit message: Added many compatibilty and fixed all issues, ready for ordering V1
Parts:
- removed C30, C52, C54, C55, C56, C58, C60, C61, C62: 10uF, Capacitor_SMD:C_0805_2012Metric
- moved U12 34.8 mm to (76.0, 57.4)
Connections:
- U1 pad 1: GND -> +3V3
Routing:
- net +3V3: track 81.4 -> 83.1 mm, vias 10 -> 11
- net GND: track 74.2 -> 73.6 mm
Other:
- board text removed: "V0.1"
