File: 4in1ESC.kicad_sch (KiCad schematic)
At the start: 62 parts, among them J1 SM08B-SRSS-TB, U1 TLV76733DRVR, U12 INA186A3IDCKR, U18 LMR51420YDDCR, U5 XRIM160808SR47MBCD

Commit message: update readme n datasheets
Parts:
- removed C30, C52, C54, C55, C56, C58, C60, C61, C62: 10uF, Capacitor_SMD:C_0805_2012Metric, symbol Device:C

Commit message: Added many compatibilty and fixed all issues, ready for ordering V1
Parts:
- U4: symbol Connector:4in1ESC -> components:4in1ESC
Changed lines of the file:
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@@
 	)
 	(symbol
-		(lib_id "Connector:4in1ESC")
+		(lib_id "components:4in1ESC")
 		(at 297.18 95.25 0)
 		(unit 1)

Commit message: Parts changes and final production files for V1
Parts:
- C10, C11, C12, C13, C14, C15, C16, C17, C18, C19, C2, C20, C21, C22, C23, C24, C25, C26, C27, C28, C29, C3, C31, C4, C40, C41, C47, C5, C51, C6, C7, C8, C9: LCSC C440198 -> C13585
Connections:
- net +3V3: now also U1.1 (OUT)
- net GND: no longer U1.1 (OUT)
