File: 4in1ESC.kicad_sch (KiCad schematic)
At the start: 53 parts, among them J1 SM08B-SRSS-TB, U1 TLV76733DRVR, U12 INA186A3IDCKR, U18 LMR51420YDDCR, U5 XRIM160808SR47MBCD

Commit message: BOM substitutions: replace OOS parts with in-stock alternatives
- 10kΩ 0201: C473048 → C106225 (Yageo RC0201FR-0710KL, 1.17M stock)
- 220Ω 0201: C473535 → C226468 (Yageo AC0201FR-07220RL, 21.9k stock)
- Ferrite bead 0201: C525479 → C440127 (Murata BLM03HD331SN1D 330Ω, 53.6k stock)
- Buck converter: C5383002 → C7296200 (LMR51420YFDDCR 1.1MHz FPWM)
- Bulk 10uF caps: C13585 → C2932476 (Samsung CL21A106KBYQNNE 0805 50V)
- Exclude test points and board outline from BOM

Co-Authored-By: Claude Opus 4.6 (1M context) <noreply@anthropic.com>
Parts:
- C10, C11, C12, C13, C14, C15, C16, C17, C18, C19, C2, C20, C21, C22, C23, C24, C25, C26, C27, C28, C29, C3, C31, C4, C40, C41, C47, C5, C51, C6, C7, C8, C9: LCSC C13585 -> C2932476
- R118: LCSC C473048 -> C106225
- U4: now left out of the parts list

Commit message: Standardize repo: .gitignore, README, license, remove production from tracking
- Standardize .gitignore to match ecosystem template
- Update README: fix production refs, add missing dirs, simplify license section
- Replace LICENSE stub with full CERN-OHL-S-2.0 text
- Remove production/ from git tracking (generated, re-exportable)
- Add previously untracked: licensing/, COST_ANALYSIS.md, tools/esc_thermal.py
- Delete NextPCB artifact (bom_template_nextpcb)

Co-Authored-By: Claude Opus 4.6 (1M context) <noreply@anthropic.com>
Parts:
- U4: value ~ -> (none)
