File: ESC.kicad_sch (KiCad schematic)
At the start: 36 parts, among them Q1 SP40N03GNJ, Q2 SP40N03GNJ, Q3 SP40N03GNJ, Q4 SP40N03GNJ, Q5 SP40N03GNJ, Q6 SP40N03GNJ, U2 AT32F421G8U7, U3 NSG2065Q

Commit message: v0.4 component swap: INA186, TLV76733, JST symbol, ferrite bead
- Replace INA199A1DCKR with INA186A3IDCKR (C2058245) current sense amp
- Replace TPS746 with TLV76733DRVR (C2848334) LDO, SNS pin wired to output
- Add SM08B-SRSS-TB and INA186A3IDCKR symbols to local library
- Add JST 3D model (CONN-SMD_SR1.00-WS-8P.step) to footprint
- Add SC-70-6 3D model for INA186
- Update ferrite bead to BLM03PX121SN1D (C525479) in ESC sub-sheet
- Schematic ready for routing, DRC errors remain to fix

Co-Authored-By: Claude Opus 4.6 <noreply@anthropic.com>
Parts:
- FB2: value 200mA -> BLM03PX121SN1D; LCSC C6132061 -> C525479
Other:
- moved on the sheet: C49, FB2
Changed lines of the file:
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@@
 	)
 	(junction
-		(at 74.93 39.37)
+		(at 74.93 35.56)
 		(diameter 0)
 		(color 0 0 0 0)
@@
 	(wire
 		(pts
-			(xy 72.39 41.91) (xy 74.93 39.37)
+			(xy 72.39 38.1) (xy 74.93 35.56)
 		)
 		(stroke
@@
 	(wire
 		(pts
-			(xy 72.39 48.26) (xy 72.39 50.8)
+			(xy 72.39 44.45) (xy 72.39 50.8)
 		)
 		(stroke
@@
 	(wire
 		(pts
-			(xy 74.93 39.37) (xy 74.93 50.8)
+			(xy 74.93 35.56) (xy 74.93 50.8)
 		)
 		(stroke
@@
 	(wire
 		(pts
-			(xy 74.93 38.1) (xy 74.93 39.37)
+			(xy 74.93 34.29) (xy 74.93 35.56)
 		)
 		(stroke
@@
 	(wire
 		(pts
-			(xy 72.39 43.18) (xy 72.39 41.91)
+			(xy 72.39 39.37) (xy 72.39 38.1)
 		)
 		(stroke
@@
 	(symbol
 		(lib_id "ESCLibrary:GRM033R61C104KE84D")
-		(at 36.83 27.94 270)
+		(at 39.37 27.94 270)
 		(unit 1)
 		(exclude_from_sim no)
@@
 		(dnp no)
 		(property "Reference" "C49"
-			(at 32.766 30.226 0)
+			(at 35.814 26.924 90)
 			(effects
 				(font
@@
 		)
 		(property "Value" "100nF"
-			(at 30.988 31.242 0)
+			(at 36.83 28.702 90)
 			(effects
 				(font
@@
 		)
 		(property "Footprint" "Capacitor_SMD:C_0201_0603Metric"
-			(at 26.67 27.94 0)
+			(at 29.21 27.94 0)
 			(effects
 				(font
@@
 		)
 		(property "Datasheet" "https://item.szlcsc.com/360022.html"
-			(at 36.957 25.654 0)
+			(at 39.497 25.654 0)
 			(effects
 				(font
@@
 		)
 		(property "Description" ""
-			(at 36.83 27.94 0)
+			(at 39.37 27.94 0)
 			(effects
 				(font
@@
 		)
 		(property "LCSC" "C181043"
-			(at 36.83 27.94 0)
+			(at 39.37 27.94 0)
 			(effects
 				(font
@@
 	)
 	(symbol
+		(lib_id "power:+3V3")
+		(at 39.37 24.13 0)
+		(unit 1)
+		(exclude_from_sim no)
+		(in_bom yes)
+		(on_board yes)
+		(dnp no)
+		(fields_autoplaced yes)
+		(property "Reference" "#PWR067"
+			(at 39.37 27.94 0)
+			(effects
+				(font
+					(size 1.27 1.27)
+				)
+				(hide yes)
+			)
+		)
+		(property "Value" "+3V3"
+			(at 39.37 19.05 0)
+			(effects
+				(font
+					(size 1.27 1.27)
+				)
+			)
+		)
+		(property "Footprint" ""
+			(at 39.37 24.13 0)
+			(effects
+				(font
+					(size 1.27 1.27)
+				)
+				(hide yes)
+			)
+		)
+		(property "Datasheet" ""
+			(at 39.37 24.13 0)
+			(effects
+				(font
+					(size 1.27 1.27)
+				)
+				(hide yes)
+			)
+		)
+		(property "Description" "Power symbol creates a global label with name \"+3V3\""
+			(at 39.37 24.13 0)
+			(effects
+				(font
+					(size 1.27 1.27)
+				)
+				(hide yes)
+			)
+		)
+		(pin "1"
+		)
+		(instances
+			(project "4in1ESC"
+				(path "/612d09d9-c556-41af-8a15-92be360f8e81/0f1ac7ef-71be-4cf4-81ac-90268323e1b3"
+					(reference "#PWR0110")
+					(unit 1)
+				)
+				(path "/612d09d9-c556-41af-8a15-92be360f8e81/3fa70197-fd52-4922-8368-62c7feb267b9"
+					(reference "#PWR088")
+					(unit 1)
+				)
+				(path "/612d09d9-c556-41af-8a15-92be360f8e81/6061fcc0-8b26-44e0-b078-a202b47fdd16"
+					(reference "#PWR0107")
+					(unit 1)
+				)
+				(path "/612d09d9-c556-41af-8a15-92be360f8e81/f870c78f-43b6-4f66-afe4-21d85c4907b1"
+					(reference "#PWR067")
+					(unit 1)
+				)
+			)
+		)
+	)
+	(symbol
 		(lib_id "ESCLibrary:0201_10kR")
 		(at 254 90.17 270)
@@
 	)
 	(symbol
-		(lib_id "power:+3V3")
-		(at 36.83 24.13 0)
-		(unit 1)
-		(exclude_from_sim no)
-		(in_bom yes)
-		(on_board yes)
-		(dnp no)
-		(fields_autoplaced yes)
-		(property "Reference" "#PWR028"
-			(at 36.83 27.94 0)
-			(effects
-				(font
-					(size 1.27 1.27)
-				)
-				(hide yes)
-			)
-		)
-		(property "Value" "+3V3"
-			(at 36.83 19.05 0)
-			(effects
-				(font
-					(size 1.27 1.27)
-				)
-			)
-		)
-		(property "Footprint" ""
-			(at 36.83 24.13 0)
-			(effects
-				(font
-					(size 1.27 1.27)
-				)
-				(hide yes)
-			)
-		)
-		(property "Datasheet" ""
-			(at 36.83 24.13 0)
-			(effects
-				(font
-					(size 1.27 1.27)
-				)
-				(hide yes)
-			)
-		)
-		(property "Description" "Power symbol creates a global label with name \"+3V3\""
-			(at 36.83 24.13 0)
-			(effects
-				(font
-					(size 1.27 1.27)
-				)
-				(hide yes)
-			)
-		)
-		(pin "1"
-		)
-		(instances
-			(project "4in1ESC"
-				(path "/612d09d9-c556-41af-8a15-92be360f8e81/0f1ac7ef-71be-4cf4-81ac-90268323e1b3"
-					(reference "#PWR088")
-					(unit 1)
-				)
-				(path "/612d09d9-c556-41af-8a15-92be360f8e81/3fa70197-fd52-4922-8368-62c7feb267b9"
-					(reference "#PWR046")
-					(unit 1)
-				)
-				(path "/612d09d9-c556-41af-8a15-92be360f8e81/6061fcc0-8b26-44e0-b078-a202b47fdd16"
-					(reference "#PWR067")
-					(unit 1)
-				)
-				(path "/612d09d9-c556-41af-8a15-92be360f8e81/f870c78f-43b6-4f66-afe4-21d85c4907b1"
-					(reference "#PWR028")
-					(unit 1)
-				)
-			)
-		)
-	)
-	(symbol
 		(lib_id "PCM_Resistor_AKL:R_0402")
 		(at 149.86 161.29 90)
@@
 	(symbol
 		(lib_id "power:+3V3")
-		(at 74.93 38.1 0)
+		(at 74.93 34.29 0)
 		(unit 1)
 		(exclude_from_sim no)
@@
 		(fields_autoplaced yes)
 		(property "Reference" "#PWR034"
-			(at 74.93 41.91 0)
+			(at 74.93 38.1 0)
 			(effects
 				(font
@@
 		)
 		(property "Value" "+3V3"
-			(at 74.93 33.02 0)
+			(at 74.93 29.21 0)
 			(effects
 				(font
@@
 		)
 		(property "Footprint" ""
-			(at 74.93 38.1 0)
+			(at 74.93 34.29 0)
 			(effects
 				(font
@@
 		)
 		(property "Datasheet" ""
-			(at 74.93 38.1 0)
+			(at 74.93 34.29 0)
 			(effects
 				(font
@@
 		)
 		(property "Description" "Power symbol creates a global label with name \"+3V3\""
-			(at 74.93 38.1 0)
+			(at 74.93 34.29 0)
 			(effects
 				(font
@@
 	(symbol
 		(lib_id "Device:FerriteBead_Small")
-		(at 72.39 45.72 0)
+		(at 72.39 41.91 0)
 		(unit 1)
 		(exclude_from_sim no)
@@
 		(fields_autoplaced yes)
 		(property "Reference" "FB2"
-			(at 74.93 44.4118 0)
+			(at 74.93 40.6018 0)
 			(effects
 				(font
@@
 			)
 		)
-		(property "Value" "200mA"
-			(at 74.93 46.9518 0)
+		(property "Value" "BLM03PX121SN1D"
+			(at 74.93 43.1418 0)
 			(effects
 				(font
@@
 		)
 		(property "Footprint" "Inductor_SMD:L_0201_0603Metric"
-			(at 70.612 45.72 90)
+			(at 70.612 41.91 90)
 			(effects
 				(font
@@
 		)
 		(property "Datasheet" "~"
-			(at 72.39 45.72 0)
+			(at 72.39 41.91 0)
 			(effects
 				(font
@@
 		)
 		(property "Description" "Ferrite bead, small symbol"
-			(at 72.39 45.72 0)
+			(at 72.39 41.91 0)
 			(effects
 				(font
@@
 			)
 		)
-		(property "LCSC" "C6132061"
-			(at 72.39 45.72 0)
+		(property "LCSC" "C525479"
+			(at 72.39 41.91 0)
 			(effects
 				(font
@@
 	(symbol
 		(lib_id "power:GND")
-		(at 36.83 31.75 0)
+		(at 39.37 31.75 0)
 		(unit 1)
 		(exclude_from_sim no)
@@
 		(dnp no)
 		(property "Reference" "#PWR029"
-			(at 36.83 38.1 0)
+			(at 39.37 38.1 0)
 			(effects
 				(font
@@
 		)
 		(property "Value" "GND"
-			(at 37.084 35.306 0)
+			(at 39.624 35.306 0)
 			(effects
 				(font
@@
 		)
 		(property "Footprint" ""
-			(at 36.83 31.75 0)
+			(at 39.37 31.75 0)
 			(effects
 				(font
@@
 		)
 		(property "Datasheet" ""
-			(at 36.83 31.75 0)
+			(at 39.37 31.75 0)
 			(effects
 				(font
@@
 		)
 		(property "Description" "Power symbol creates a global label with name \"GND\" , ground"
-			(at 36.83 31.75 0)
+			(at 39.37 31.75 0)
 			(effects
 				(font

Commit message: BOM substitutions: replace OOS parts with in-stock alternatives
- 10kΩ 0201: C473048 → C106225 (Yageo RC0201FR-0710KL, 1.17M stock)
- 220Ω 0201: C473535 → C226468 (Yageo AC0201FR-07220RL, 21.9k stock)
- Ferrite bead 0201: C525479 → C440127 (Murata BLM03HD331SN1D 330Ω, 53.6k stock)
- Buck converter: C5383002 → C7296200 (LMR51420YFDDCR 1.1MHz FPWM)
- Bulk 10uF caps: C13585 → C2932476 (Samsung CL21A106KBYQNNE 0805 50V)
- Exclude test points and board outline from BOM

Co-Authored-By: Claude Opus 4.6 (1M context) <noreply@anthropic.com>
Parts:
- FB2: value BLM03PX121SN1D -> BLM03HD331SN1D; LCSC C525479 -> C440127
- R18, R19, R25, R27, R28, R30, R31, R33: LCSC C473048 -> C106225
- R20: LCSC C473535 -> C226468
- TP1, TP4: now left out of the parts list
Changed lines of the file:
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@@
 			)
 		)
-		(property "LCSC" "C473048"
+		(property "LCSC" "C106225"
 			(at 234.95 99.06 0)
 			(effects
@@
 		(unit 1)
 		(exclude_from_sim no)
-		(in_bom yes)
+		(in_bom no)
 		(on_board yes)
 		(dnp no)
@@
 			)
 		)
-		(property "LCSC" "C473048"
+		(property "LCSC" "C106225"
 			(at 205.74 90.17 0)
 			(effects
@@
 			)
 		)
-		(property "LCSC" "C473048"
+		(property "LCSC" "C106225"
 			(at 210.82 99.06 0)
 			(effects
@@
 			)
 		)
-		(property "LCSC" "C473048"
+		(property "LCSC" "C106225"
 			(at 49.53 60.96 0)
 			(effects
@@
 			)
 		)
-		(property "LCSC" "C473048"
+		(property "LCSC" "C106225"
 			(at 259.08 99.06 0)
 			(effects
@@
 			)
 		)
-		(property "LCSC" "C473048"
+		(property "LCSC" "C106225"
 			(at 254 90.17 0)
 			(effects
@@
 			)
 		)
-		(property "LCSC" "C473048"
+		(property "LCSC" "C106225"
 			(at 229.87 90.17 0)
 			(effects
@@
 			)
 		)
-		(property "Value" "BLM03PX121SN1D"
+		(property "Value" "BLM03HD331SN1D"
 			(at 74.93 43.1418 0)
 			(effects
@@
 			)
 		)
-		(property "LCSC" "C525479"
+		(property "LCSC" "C440127"
 			(at 72.39 41.91 0)
 			(effects
@@
 			)
 		)
-		(property "LCSC" "C473535"
+		(property "LCSC" "C226468"
 			(at 49.53 80.01 0)
 			(effects
@@
 		(unit 1)
 		(exclude_from_sim no)
-		(in_bom yes)
+		(in_bom no)
 		(on_board yes)
 		(dnp no)
@@
 			)
 		)
-		(property "LCSC" "C473048"
+		(property "LCSC" "C106225"
 			(at 34.29 63.5 0)
 			(effects
